Commit message: 增加了obj文件

File: urdf/myurdf_fix.urdf (robot description, URDF)
Before this commit: robot myurdf_fix, 9 links, 8 joints
Links:
- link back_left_steering: geometry collision mesh filename=package://myurdf_fix/meshes/back_left_steering.obj; visual mesh filename=package://myurdf_fix/meshes/back_left_steering.obj
- link back_left_wheel: geometry collision mesh filename=package://myurdf_fix/meshes/back_left_wheel.obj; visual mesh filename=package://myurdf_fix/meshes/back_left_wheel.obj
- link back_right_steering: geometry collision mesh filename=package://myurdf_fix/meshes/back_right_steering.obj; visual mesh filename=package://myurdf_fix/meshes/back_right_steering.obj
- link back_right_wheel: geometry collision mesh filename=package://myurdf_fix/meshes/back_right_wheel.obj; visual mesh filename=package://myurdf_fix/meshes/back_right_wheel.obj
- link base_link: geometry collision mesh filename=package://myurdf_fix/meshes/base_link.obj; visual mesh filename=package://myurdf_fix/meshes/base_link.obj
- link front_left_steering: geometry collision mesh filename=package://myurdf_fix/meshes/front_left_steering.obj; visual mesh filename=package://myurdf_fix/meshes/front_left_steering.obj
- link front_left_wheel: geometry collision mesh filename=package://myurdf_fix/meshes/front_left_wheel.obj; visual mesh filename=package://myurdf_fix/meshes/front_left_wheel.obj
- link front_right_steering: geometry collision mesh filename=package://myurdf_fix/meshes/front_right_steering.obj; visual mesh filename=package://myurdf_fix/meshes/front_right_steering.obj
- link front_right_wheel: geometry collision mesh filename=package://myurdf_fix/meshes/front_right_wheel.obj; visual mesh filename=package://myurdf_fix/meshes/front_right_wheel.obj

Commit message: 更改urdf

File: urdf/myurdf_fix.urdf (robot description, URDF)
Before this commit: robot myurdf_fix, 9 links, 8 joints
Links:
- added link base_footprint
- added link camera_link
- added link laser_link
Joints:
- added joint base_footprint_joint: type None, parent base_footprint, child base_link, origin xyz=0 0 0 rpy=0 0 0
- added joint camera_joint: type None, parent base_link, child camera_link, origin xyz=0 0 0.15 rpy=0 0 0
- added joint laser_joint: type None, parent base_link, child laser_link, origin xyz=0 0 0.15 rpy=0 0 0

Commit message: fix add camera laser

File: urdf/myurdf_fix.urdf (robot description, URDF)
Before this commit: robot myurdf_fix, 12 links, 11 joints
Joints:
- joint base_footprint_joint: type None -> fixed
- joint camera_joint: type None -> fixed
- joint laser_joint: origin xyz=0 0 0.15 rpy=0 0 0 -> xyz=0 0 0.4 rpy=0 0 3.1415926; type None -> fixed

Commit message: 更换了camera与laser的坐标

File: urdf/myurdf_fix.urdf (robot description, URDF)
Before this commit: robot myurdf_fix, 12 links, 11 joints
Joints:
- joint camera_joint: origin xyz=0 0 0.15 rpy=0 0 0 -> xyz=0 0 0.4 rpy=0 0 3.1415926
- joint laser_joint: origin xyz=0 0 0.4 rpy=0 0 3.1415926 -> xyz=0 0 0.15 rpy=0 0 0
